File: MP3/Liam Eclectronics MP3.kicad_pcb (KiCad board)
At the start: 2 copper layers, 52.4 x 57.7 mm, 43 parts, among them J1 USB4105-GF-A, J4 DEBUG, J5 Conn_01x10, J6 Conn_01x10, J7 Conn_01x10, J8 Conn_01x10, U1 RP2354A, U2 MCP1702T-3302E_CB, X1 IQXO-791_12MHz

Commit message: some small fixes
Routing:
- net +3V3: vias 1 -> 0
Changed lines of the file:
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@@
 		(end 143.55 56.7)
 		(stroke
-			(width 0.3048)
+			(width 0.2032)
 			(type solid)
 		)
@@
 		(net "+3V3")
 	)
-	(via
-		(at 136.1 85.425)
-		(size 0.6096)
-		(drill 0.3048)
-		(layers "F.Cu" "B.Cu")
-		(free yes)
-		(net "+3V3")
-	)
