File: MP3/Liam Eclectronics MP3.kicad_pcb (KiCad board)
At the start: 2 copper layers, 52.4 x 57.7 mm, 43 parts, among them J1 USB4105-GF-A, J4 DEBUG, J5 Conn_01x10, J6 Conn_01x10, J7 Conn_01x10, J8 Conn_01x10, U1 RP2354A, U2 MCP1702T-3302E_CB, X1 IQXO-791_12MHz

Commit message: minor fixes
Routing:
- net +5V: track 3.06 -> 1.59 mm
Other:
- board text added: "GPIO0"
Changed lines of the file:
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@@
 		(tags "Through hole pin header THT 1x10 2.54mm single row")
 		(property "Reference" "J5"
-			(at 0 -2.38 0)
+			(at 0.025 -3.015 0)
 			(layer "F.SilkS")
 			(effects
@@
 	(gr_poly
 		(pts
+			(xy 134.575 44.9) (xy 135.075 44.9) (xy 135.075 43.989286) (xy 135.825 43.560714) (xy 135.825 43.425)
+			(xy 134.986957 43.425) (xy 134.963142 43.972757) (xy 134.575 44.250001)
+		)
+		(stroke
+			(width 0.2)
+			(type solid)
+		)
+		(fill yes)
+		(layer "F.Cu")
+		(net "+5V")
+	)
+	(gr_poly
+		(pts
 			(xy 138.2 51.35) (xy 137.01226 51.347135) (xy 137 49.8) (xy 137.45 48.35) (xy 139.05 48.35) (xy 139.05 49.1)
 			(xy 139.05 49.55) (xy 138.8 49.8) (xy 138.8 50.75) (xy 138.3 50.75)
@@
 	)
 	(gr_text "PWM Pref"
-		(at 122.525 56.8 0)
+		(at 120.875 57.225 0)
 		(layer "F.SilkS")
 		(effects
 			(font
-				(size 0.381 0.381)
-				(thickness 0.09525)
+				(size 0.762 0.6096)
+				(thickness 0.1524)
 				(bold yes)
 			)
@@
 	)
 	(gr_text "PWM Pref"
-		(at 127.7 71.125 0)
+		(at 127.05 71.175 0)
 		(layer "F.SilkS")
 		(effects
 			(font
-				(size 0.381 0.381)
-				(thickness 0.09525)
+				(size 0.762 0.6096)
+				(thickness 0.1524)
 				(bold yes)
 			)
@@
 	)
 	(gr_text "ADC"
-		(at 150.6 56.525 0)
+		(at 150.55 56.9 0)
 		(layer "F.SilkS")
 		(effects
 			(font
-				(size 0.381 0.381)
-				(thickness 0.09525)
+				(size 0.762 0.6096)
+				(thickness 0.1524)
 				(bold yes)
 			)
@@
 	)
 	(gr_text "ADC"
-		(at 150.6 66.675 0)
+		(at 152.875 62.125 0)
 		(layer "F.SilkS")
 		(effects
 			(font
-				(size 0.381 0.381)
-				(thickness 0.09525)
+				(size 0.762 0.6096)
+				(thickness 0.1524)
 				(bold yes)
 			)
@@
 	)
 	(gr_text "ADC"
-		(at 153.425 57.1 0)
+		(at 153.1 57.1 0)
 		(layer "F.SilkS")
 		(effects
 			(font
-				(size 0.381 0.381)
-				(thickness 0.09525)
+				(size 0.762 0.6096)
+				(thickness 0.1524)
 				(bold yes)
 			)
@@
 	)
 	(gr_text "ADC"
-		(at 153.525 62.025 0)
+		(at 150.55 67 0)
 		(layer "F.SilkS")
 		(effects
 			(font
-				(size 0.381 0.381)
-				(thickness 0.09525)
+				(size 0.6096 0.762)
+				(thickness 0.1524)
 				(bold yes)
 			)
@@
 		)
 	)
+	(gr_text "GPIO0"
+		(at 127.95 43.525 0)
+		(layer "F.SilkS")
+		(effects
+			(font
+				(size 0.762 0.762)
+				(thickness 0.1524)
+				(bold yes)
+			)
+			(justify left bottom)
+		)
+	)
 	(gr_text "GND"
 		(at 129.75 76.875 0)
@@
 	)
 	(segment
-		(start 134.83 44.122514)
-		(end 135.0206 43.931914)
-		(width 0.4572)
-		(layer "F.Cu")
-		(net "+5V")
-	)
-	(segment
-		(start 135.0206 43.931914)
-		(end 135.0206 43.7294)
-		(width 0.4572)
-		(layer "F.Cu")
-		(net "+5V")
-	)
-	(segment
-		(start 134.83 44.725)
-		(end 134.83 44.122514)
-		(width 0.4572)
-		(layer "F.Cu")
-		(net "+5V")
-	)
-	(segment
 		(start 143.2 39.35)
 		(end 143.8 39.35)
@@
 		(layer "F.Cu")
 		(net "+5V")
-	)
-	(segment
-		(start 135.0206 43.7294)
-		(end 135.3 43.45)
-		(width 0.4572)
-		(layer "F.Cu")
-		(net "+5V")
